Commit message: add custom_display

File: ur5e_2f_85/ur5e_2f_85_description/urdf/ur5e_2f_85_macro.xacro (robot description, xacro)
@@ -14,4 +14,5 @@
         use_fake_hardware
         com_port">
+        <link name="tcp_link"/>
         <xacro:ur_robot
             name="${name}"
@@ -36,4 +37,9 @@
             <origin xyz="0 0 0" rpy="0 0 0" />
         </xacro:robotiq_gripper>
+        <joint name="joint_tcp" type="fixed">
+            <parent link="tool0"/>
+            <child link="tcp_link"/>
+            <origin xyz="0 0 0.147" rpy="0 0 0"/>
+        </joint>
     </xacro:macro>
 </robot>
