Commit message: gripper integration pt. 1

File: ur5e_2f_85/ur5e_2f_85_description/urdf/ur5e_2f_85_platform.urdf (robot description, URDF)
Before this commit: robot ur5e_2f_85, 39 links, 38 joints
Links:
- added link ur_mount_link
- link adapter_gripper: geometry 
- link base: geometry 
- link base_link: geometry 
- link ft_frame: geometry 
- link tcp_link: geometry 
- link tool0: geometry 
- link world: geometry 
Joints:
- added joint ur_mount_joint: type fixed, parent robot_base_1, child ur_mount_link, origin xyz=0 0 0 rpy=0 0 3.14159265359
- joint base_joint: parent robot_base_1 -> ur_mount_link

File: ur5e_2f_85/ur5e_2f_85_description/urdf/ur5e_2f_85_platform.urdf.xacro (robot description, xacro)
@@ -25,8 +25,14 @@
         <link name="$(arg parent)"/>
         <xacro:robot_platform parent="$(arg parent)"/>
+        <link name="ur_mount_link"/>
+        <joint name="ur_mount_joint" type="fixed">
+        <parent link="robot_base_1"/>
+        <child  link="ur_mount_link"/>
+        <origin xyz="0 0 0" rpy="0 0 3.14159265359"/>
+        </joint>
         <xacro:ur5e_2f_85
             name="$(arg name)"
             tf_prefix="$(arg tf_prefix)"
-            parent="robot_base_1"
+            parent="ur_mount_link"
             joint_limit_params="$(arg joint_limit_params)"
             kinematics_params="$(arg kinematics_params)"

File: ur5e_2f_85/ur5e_2f_85_description/urdf/ur5e_2f_85_platform_control.urdf.xacro (robot description, xacro)
@@ -20,6 +20,6 @@
     <xacro:arg name="safety_pos_margin" default="0.15"/>
     <xacro:arg name="safety_k_position" default="20"/>
-    <xacro:arg name="use_fake_hardware" default="true" />
-    <xacro:arg name="com_port" default="/dev/ttyUSB0" />
+    <xacro:arg name="use_fake_hardware" default="false" />
+    <xacro:arg name="com_port" default="/tmp/ttyUR" />
     <xacro:arg name="parent" default="world" />
     <xacro:arg name="force_abs_paths" default="false" />
@@ -57,8 +57,14 @@
         <link name="$(arg parent)"/>
         <xacro:robot_platform parent="$(arg parent)"/>
+        <link name="ur_mount_link"/>
+        <joint name="ur_mount_joint" type="fixed">
+        <parent link="robot_base_1"/>
+        <child  link="ur_mount_link"/>
+        <origin xyz="0 0 0" rpy="0 0 3.14159265359"/>
+        </joint>
         <xacro:ur5e_2f_85
             name="$(arg name)"
             tf_prefix="$(arg tf_prefix)"
-            parent="robot_base_1"
+            parent="ur_mount_link"
             joint_limit_params="$(arg joint_limit_params)"
             kinematics_params="$(arg kinematics_params)"
