Commit message: Modified for isaac integration

File: ur5e_2f_85/ur5e_2f_85_description/urdf/ur5e_2f_85_platform.urdf (robot description, URDF)
Before this commit: robot ur5e_2f_85, 40 links, 39 joints
Links:
- removed link zed_camera
- removed link zed_mini_camera_attach_back_base_with_external_rack
- added link zed_mini_camera_center; collision mesh filename=package://zed_description/meshes/zedm.stl; visual mesh filename=package://zed_description/meshes/zedm.stl
- added link zed_mini_camera_link
- added link zed_mini_left_camera_frame
- added link zed_mini_left_camera_frame_optical
- added link zed_mini_right_camera_frame
- added link zed_mini_right_camera_frame_optical
Joints:
- removed joint camera_attach
- added joint zed_mini_camera_center_joint: type fixed, parent zed_mini_camera_link, child zed_mini_camera_center, origin xyz=0 0 0.01325 rpy=0 0.0 0
- added joint zed_mini_left_camera_joint: type fixed, parent zed_mini_camera_center, child zed_mini_left_camera_frame, origin xyz=0.0 0.0315 0 rpy=0 0 0
- added joint zed_mini_left_camera_optical_joint: type fixed, parent zed_mini_left_camera_frame, child zed_mini_left_camera_frame_optical, origin xyz=0 0 0 rpy=-1.5707963267948966 0.0 -1.5707963267948966
- added joint zed_mini_right_camera_joint: type fixed, parent zed_mini_camera_center, child zed_mini_right_camera_frame, origin xyz=0.0 -0.0315 0 rpy=0 0 0
- added joint zed_mini_right_camera_optical_joint: type fixed, parent zed_mini_right_camera_frame, child zed_mini_right_camera_frame_optical, origin xyz=0 0 0 rpy=-1.5707963267948966 0.0 -1.5707963267948966
- joint base_link_camera_attach: origin xyz=0.0 0.0 0.0 rpy=0 0 0 -> xyz=0.0 0.008 -0.0105 rpy=0 0 0
- joint camera_base: child zed_camera -> zed_mini_camera_link; origin xyz=0.008 0.011954 -0.000301 rpy=0 0 0 -> xyz=-0.008 0.0460 0.007 rpy=-1.5708  -1.5708 0; parent zed_mini_camera_attach_back_base_with_external_rack -> upper_block_gripper
- joint robotiq_85_left_finger_tip_joint: limit (none) -> lower=-0.8 upper=0.0 effort=50 velocity=0.5; type continuous -> revolute
- joint robotiq_85_left_inner_knuckle_joint: limit (none) -> lower=0.0 upper=0.8 effort=50 velocity=0.5; type continuous -> revolute
- joint robotiq_85_right_finger_tip_joint: limit (none) -> lower=0.0 upper=0.8 effort=50 velocity=0.5; type continuous -> revolute
- joint robotiq_85_right_inner_knuckle_joint: limit (none) -> lower=-0.8 upper=0.0 effort=50 velocity=0.5; type continuous -> revolute
