Commit message: update camera urdf

File: ur5e_2f_85/ur5e_2f_85_description/urdf/zed_mini_camera_macro.xacro (robot description, xacro)
@@ -1,4 +1,7 @@
 <?xml version="1.0"?>
 <robot xmlns:xacro="http://wiki.ros.org/xacro">
+  <!-- official Stereolabs ZED Mini model (mesh + optical frames), see
+       zed_description package (cloned from stereolabs/zed-ros2-description) -->
+  <xacro:include filename="$(find zed_description)/urdf/zed_macro.urdf.xacro"/>
   <xacro:macro name="camera_gripper_attach" params="parent prefix">
     <joint name="${prefix}camera_attach_joint" type="fixed">
@@ -27,5 +30,5 @@
     <link name="${prefix}upper_block_gripper">
       <visual>
-        <origin xyz="0.0 -0.0 -0.0" rpy="0 0 0"/>
+        <origin xyz="0.0 -0.0 -0.0" rpy="0 0 1.5708"/>
         <geometry>
           <mesh filename="package://ur5e_2f_85_description/meshes/camera_gripper_attach/upper_block_gripper.stl" scale="0.001 0.001 0.001"/>
@@ -34,5 +37,5 @@
       </visual>
       <collision>
-        <origin xyz="0.0 -0.0 -0.0" rpy="0 0 0"/>
+        <origin xyz="0.0 -0.0 -0.0" rpy="0 0 1.5708"/>
         <geometry>
           <mesh filename="package://ur5e_2f_85_description/meshes/camera_gripper_attach/upper_block_gripper.stl" scale="0.001 0.001 0.001"/>
@@ -40,5 +43,5 @@
       </collision>
     </link>
-    <link name="${prefix}zed_mini_camera_attach_back_base_with_external_rack">
+    <!-- <link name="${prefix}zed_mini_camera_attach_back_base_with_external_rack">
       <visual>
         <origin xyz="-4e-05 -0.08901 -0.0" rpy="0 0 0"/>
@@ -54,35 +57,30 @@
         </geometry>
       </collision>
-    </link>
-    <link name="${prefix}zed_camera">
-      <visual>
-        <origin xyz="-0.00804 -0.100964 0.000301" rpy="0 0 0"/>
-        <geometry>
-          <mesh filename="package://ur5e_2f_85_description/meshes/camera_gripper_attach/zed_camera.stl" scale="0.001 0.001 0.001"/>
-        </geometry>
-        <material name="silver_camera"/>
-      </visual>
-      <collision>
-        <origin xyz="-0.00804 -0.100964 0.000301" rpy="0 0 0"/>
-        <geometry>
-          <mesh filename="package://ur5e_2f_85_description/meshes/camera_gripper_attach/zed_camera.stl" scale="0.001 0.001 0.001"/>
-        </geometry>
-      </collision>
-    </link>
+    </link> -->
     <joint name="${prefix}base_link_camera_attach" type="fixed">
-      <origin xyz="0.0 0.0 0.0" rpy="0 0 0"/>
+      <origin xyz="0.0 0.008 -0.0105" rpy="0 0 0"/>
       <parent link="${prefix}base_link_camera"/>
       <child link="${prefix}upper_block_gripper"/>
     </joint>
-    <joint name="${prefix}camera_attach" type="fixed">
+    <!-- <joint name="${prefix}camera_attach" type="fixed">
       <origin xyz="4e-05 0.08901 0.0" rpy="0 0 0"/>
       <parent link="${prefix}upper_block_gripper"/>
       <child link="${prefix}zed_mini_camera_attach_back_base_with_external_rack"/>
+    </joint> -->
+    <!-- origin computed so the zedm.stl body mesh's bounding-box center
+         coincides with upper_block_gripper.stl's bounding-box center
+         (both expressed in the upper_block_gripper link frame), i.e. the
+         camera is centered in the rack instead of matching the old custom
+         zed_camera.stl mesh's own coordinate convention -->
+    <joint name="${prefix}camera_base" type="fixed">
+      <origin xyz="-0.008 0.0460 0.007" rpy="-1.5708  -1.5708 0"/>
+      <parent link="${prefix}upper_block_gripper"/>
+      <child link="${prefix}zed_mini_camera_link"/>
     </joint>
-    <joint name="${prefix}camera_base" type="fixed">
-      <origin xyz="0.008 0.011954 -0.000301" rpy="0 0 0"/>
-      <parent link="${prefix}zed_mini_camera_attach_back_base_with_external_rack"/>
-      <child link="${prefix}zed_camera"/>
-    </joint>
+    <!-- official ZED Mini model, attached at ${prefix}zed_mini_camera_link
+         (the mount point created by the zed_camera macro above) -->
+    <xacro:zed_camera name="${prefix}zed_mini" model="zedm">
+      <origin xyz="0 0 0" rpy="0 0 0"/>
+    </xacro:zed_camera>
   </xacro:macro>
 </robot>
