Commit message: bug fix in loading description

File: ur5e_2f_85/ur5e_2f_85_description/urdf/ur5e_2f_85_platform_control.urdf.xacro (robot description, xacro)
@@ -53,4 +53,12 @@
     <!-- convert to property to use substitution in function -->
     <xacro:property name="initial_positions_file" default="$(arg initial_positions_file)"/>
+    <!-- initial_positions_file is a global xacro:arg shared with other entry
+         points (e.g. ur5e_2f_85_moveit_config's ur5e_2f_85.urdf.xacro), whose
+         own initial_positions.yaml wraps the joint map under an
+         'initial_positions:' key (MoveIt Setup Assistant convention), unlike
+         the stock ur_description one which is a flat joint map. Normalize
+         both shapes here instead of assuming one. -->
+    <xacro:property name="initial_positions_raw" value="${xacro.load_yaml(initial_positions_file)}"/>
+    <xacro:property name="initial_positions_yaml" value="${initial_positions_raw['initial_positions'] if 'initial_positions' in initial_positions_raw else initial_positions_raw}"/>
     <xacro:macro name="ur5e_2f_85_with_platform">
         <!-- Create world link-->
@@ -85,5 +93,5 @@
         mock_sensor_commands="$(arg mock_sensor_commands)"
         headless_mode="$(arg headless_mode)"
-        initial_positions="${xacro.load_yaml(initial_positions_file)}"
+        initial_positions="${initial_positions_yaml}"
         use_tool_communication="$(arg use_tool_communication)"
         tool_voltage="$(arg tool_voltage)"
