Commit message: Complete Isaac Sim integration for SeeDo

File: ur5e_2f_85/ur5e_2f_85_moveit_config/config/ur5e_2f_85.isaac.urdf.xacro (robot description, xacro)
@@ -3,5 +3,5 @@
     <xacro:arg
         name="initial_positions_file"
-        default="initial_positions.yaml" />
+        default="initial_positions_isaac.yaml" />
     <!-- Same robot description used by the existing MoveIt config -->
     <xacro:include

File: ur5e_2f_85/ur5e_2f_85_moveit_config/config/ur5e_2f_85.isaac_ros2_control.xacro (robot description, xacro)
@@ -61,4 +61,11 @@
                 <state_interface name="velocity"/>
             </joint>
+            <joint name="robotiq_85_left_knuckle_joint">
+                <command_interface name="position"/>
+                <state_interface name="position">
+                    <param name="initial_value">0.0</param>
+                </state_interface>
+                <state_interface name="velocity"/>
+            </joint>
         </ros2_control>
     </xacro:macro>
